Commit message: working good

File: src/perrobot_description/urdf/gazebo.xacro (robot description, xacro)
@@ -1,3 +1,3 @@
-<?xml version="1.0"?>
+<?xml version="10.0"?>
 <robot xmlns:xacro="http://playerstage.sourceforge.net/gazebo/xmlschema/#interface" name="perrobot">
   <gazebo>
@@ -95,31 +95,210 @@
         </actuator>
     </transmission>
-  <gazebo reference="FL_KFE">
-    <mu1>1.0</mu1>
-    <mu2>1.0</mu2>
-    <minDepth>0.0002</minDepth>
-    <kp  value="1000000.0"/>
-    <kd  value="100.0"/>
-  </gazebo>
-  <gazebo reference="HL_KFE">
-    <mu1>1.0</mu1>
-    <mu2>1.0</mu2>
-    <minDepth>0.0002</minDepth>
-    <kp  value="1000000.0"/>
-    <kd  value="100.0"/>
-  </gazebo>
-  <gazebo reference="FR_KFE">
-    <mu1>1.0</mu1>
-    <mu2>1.0</mu2>
-    <minDepth>0.0002</minDepth>
-    <kp  value="1000000.0"/>
-    <kd  value="100.0"/>
-  </gazebo>
-  <gazebo reference="HR_KFE">
-    <mu1>1.0</mu1>
-    <mu2>1.0</mu2>
-    <minDepth>0.0002</minDepth>
-    <kp  value="1000000.0"/>
-    <kd  value="100.0"/>
-  </gazebo>
+   <gazebo reference="base_link">
+        <collision>
+            <surface>
+                <friction>
+                    <ode>
+                        <mu>1.0</mu>
+                        <mu2>1.0</mu2>
+                    </ode>
+                </friction>
+                <bounce>
+                    <restitution_coefficient>0.0</restitution_coefficient>
+                    <threshold>0.01</threshold>
+                </bounce>
+                <contact>
+                    <ode>
+                        <kp>1e5</kp>
+                        <max_vel>0.01</max_vel>
+                        <min_depth>0.001</min_depth>
+                    </ode>
+                </contact>
+            </surface>
+        </collision>
+    </gazebo>
+    <gazebo reference="FL_UPPER_LEG">
+        <collision>
+            <surface>
+                <friction>
+                    <ode>
+                        <mu>1.0</mu>
+                        <mu2>1.0</mu2>
+                    </ode>
+                </friction>
+                <bounce>
+                    <restitution_coefficient>0.0</restitution_coefficient>
+                    <threshold>0.01</threshold>
+                </bounce>
+                <contact>
+                    <ode>
+                        <kp>1e5</kp>
+                        <max_vel>0.01</max_vel>
+                        <min_depth>0.001</min_depth>
+                    </ode>
+                </contact>
+            </surface>
+        </collision>
+    </gazebo>
+    <gazebo reference="FL_LOWER_LEG">
+        <collision>
+            <surface>
+                <friction>
+                    <ode>
+                        <mu>1.0</mu>
+                        <mu2>1.0</mu2>
+                    </ode>
+                </friction>
+                <bounce>
+                    <restitution_coefficient>0.0</restitution_coefficient>
+                    <threshold>0.01</threshold>
+                </bounce>
+                <contact>
+                    <ode>
+                        <kp>1e5</kp>
+                        <max_vel>0.01</max_vel>
+                        <min_depth>0.001</min_depth>
+                    </ode>
+                </contact>
+            </surface>
+        </collision>
+    </gazebo>
+    <gazebo reference="FR_UPPER_LEG">
+        <collision>
+            <surface>
+                <friction>
+                    <ode>
+                        <mu>1.0</mu>
+                        <mu2>1.0</mu2>
+                    </ode>
+                </friction>
+                <bounce>
+                    <restitution_coefficient>0.0</restitution_coefficient>
+                    <threshold>0.01</threshold>
+                </bounce>
+                <contact>
+                    <ode>
+                        <kp>1e5</kp>
+                        <max_vel>0.01</max_vel>
+                        <min_depth>0.001</min_depth>
+                    </ode>
+                </contact>
+            </surface>
+        </collision>
+    </gazebo>
+    <gazebo reference="FR_LOWER_LEG">
+        <collision>
+            <surface>
+                <friction>
+                    <ode>
+                        <mu>1.0</mu>
+                        <mu2>1.0</mu2>
+                    </ode>
+                </friction>
+                <bounce>
+                    <restitution_coefficient>0.0</restitution_coefficient>
+                    <threshold>0.01</threshold>
+                </bounce>
+                <contact>
+                    <ode>
+                        <kp>1e5</kp>
+                        <max_vel>0.01</max_vel>
+                        <min_depth>0.001</min_depth>
+                    </ode>
+                </contact>
+            </surface>
+        </collision>
+    </gazebo>
+    <gazebo reference="HL_UPPER_LEG">
+        <collision>
+            <surface>
+                <friction>
+                    <ode>
+                        <mu>1.0</mu>
+                        <mu2>1.0</mu2>
+                    </ode>
+                </friction>
+                <bounce>
+                    <restitution_coefficient>0.0</restitution_coefficient>
+                    <threshold>0.01</threshold>
+                </bounce>
+                <contact>
+                    <ode>
+                        <kp>1e5</kp>
+                        <max_vel>0.01</max_vel>
+                        <min_depth>0.001</min_depth>
+                    </ode>
+                </contact>
+            </surface>
+        </collision>
+    </gazebo>
+    <gazebo reference="HL_LOWER_LEG">
+        <collision>
+            <surface>
+                <friction>
+                    <ode>
+                        <mu>1.0</mu>
+                        <mu2>1.0</mu2>
+                    </ode>
+                </friction>
+                <bounce>
+                    <restitution_coefficient>0.0</restitution_coefficient>
+                    <threshold>0.01</threshold>
+                </bounce>
+                <contact>
+                    <ode>
+                        <kp>1e5</kp>
+                        <max_vel>0.01</max_vel>
+                        <min_depth>0.001</min_depth>
+                    </ode>
+                </contact>
+            </surface>
+        </collision>
+    </gazebo>
+<gazebo reference="HR_UPPER_LEG">
+        <collision>
+            <surface>
+                <friction>
+                    <ode>
+                        <mu>1.0</mu>
+                        <mu2>1.0</mu2>
+                    </ode>
+                </friction>
+                <bounce>
+                    <restitution_coefficient>0.0</restitution_coefficient>
+                    <threshold>0.01</threshold>
+                </bounce>
+                <contact>
+                    <ode>
+                        <kp>1e5</kp>
+                        <max_vel>0.01</max_vel>
+                        <min_depth>0.001</min_depth>
+                    </ode>
+                </contact>
+            </surface>
+        </collision>
+    </gazebo>
+    <gazebo reference="HR_LOWER_LEG">
+        <collision>
+            <surface>
+                <friction>
+                    <ode>
+                        <mu>1.0</mu>
+                        <mu2>1.0</mu2>
+                    </ode>
+                </friction>
+                <bounce>
+                    <restitution_coefficient>0.0</restitution_coefficient>
+                    <threshold>0.01</threshold>
+                </bounce>
+                <contact>
+                    <ode>
+                        <kp>1e5</kp>
+                        <max_vel>0.01</max_vel>
+                        <min_depth>0.001</min_depth>
+                    </ode>
+                </contact>
+            </surface>
+        </collision>
+    </gazebo>
 </robot>

File: src/perrobot_description/urdf/leg.xacro (robot description, xacro)
@@ -13,4 +13,5 @@
   <xacro:property name="KFE_2_FOOT_y" value="${9.0 * 0.001}" />
   <xacro:property name="KFE_2_FOOT_z" value="${160.00 * 0.001}" />
+  <xacro:property name="effort_limit" value="1.4" />
   <!-- Macro defining solo leg. -->
   <xacro:macro name="leg" params="prefix is_front is_right has_side_motion
@@ -20,5 +21,5 @@
         <parent link="base_link"/>
         <child link="${prefix}_SHOULDER"/>
-        <limit effort="1000" lower="-10" upper="10" velocity="1000"/>
+        <limit effort="${effort_limit}" lower="-10" upper="10" velocity="1000"/>
         <!-- joints rotates around the x-axis -->
         <axis xyz="1 0 0"/>
@@ -151,5 +152,5 @@
         <parent link="${prefix}_SHOULDER"/>
         <child link="${prefix}_UPPER_LEG"/>
-        <limit effort="1000" lower="-10" upper="10" velocity="1000"/>
+        <limit effort="${effort_limit}" lower="-10" upper="10" velocity="1000"/>
         <!-- joints rotates around the y-axis -->
         <axis xyz="0 1 0"/>
@@ -180,5 +181,5 @@
         <parent link="base_link"/>
         <child link="${prefix}_UPPER_LEG"/>
-        <limit effort="1000" lower="-10" upper="10" velocity="1000"/>
+        <limit effort="${effort_limit}" lower="-10" upper="10" velocity="1000"/>
         <!-- joints rotates around the y-axis -->
         <axis xyz="0 1 0"/>
@@ -266,5 +267,5 @@
       <parent link="${prefix}_UPPER_LEG"/>
       <child link="${prefix}_LOWER_LEG"/>
-      <limit effort="1000" lower="-10" upper="10" velocity="1000"/>
+      <limit effort="${effort_limit}" lower="-10" upper="10" velocity="1000"/>
       <!-- joints rotates around the y-axis -->
       <axis xyz="0 1 0"/>
@@ -361,5 +362,5 @@
       </xacro:if>
       <!-- Limits -->
-      <limit effort="1000" lower="-10" upper="10" velocity="1000"/>
+      <limit effort="${effort_limit}" lower="-10" upper="10" velocity="1000"/>
       <!-- pybullet simulation parameters -->
       <dynamics damping="0.0" friction="0.0"/>
