Commit message: all ok exp. movement backward

File: src/perrobot_description/urdf/gazebo.xacro (robot description, xacro)
@@ -96,21 +96,26 @@
     </transmission>
    <gazebo reference="base_link">
-        <collision>
-            <surface>
-                <friction>
-                    <ode>
-                        <mu>1.0</mu>
-                        <mu2>1.0</mu2>
-                    </ode>
-                </friction>
-                <bounce>
-                    <restitution_coefficient>0.0</restitution_coefficient>
-                    <threshold>0.01</threshold>
-                </bounce>
-                <contact>
-                    <ode>
-                        <kp>1e5</kp>
-                        <max_vel>0.01</max_vel>
-                        <min_depth>0.001</min_depth>
+        <visual>
+            <material name="Black">
+                <color rgba="1.0 1.0 1.0 1.0"/>
+            </material>
+        </visual>
+        <collision>
+            <surface>
+                <friction>
+                    <ode>
+                        <mu>1.0</mu>
+                        <mu2>1.0</mu2>
+                    </ode>
+                </friction>
+                <bounce>
+                    <restitution_coefficient>0.0</restitution_coefficient>
+                    <threshold>0.01</threshold>
+                </bounce>
+                <contact>
+                    <ode>
+                        <kp>1e5</kp>
+                        <max_vel>0.1</max_vel>
+                        <min_depth>0.002</min_depth>
                     </ode>
                 </contact>
@@ -119,21 +124,26 @@
     </gazebo>
     <gazebo reference="FL_UPPER_LEG">
-        <collision>
-            <surface>
-                <friction>
-                    <ode>
-                        <mu>1.0</mu>
-                        <mu2>1.0</mu2>
-                    </ode>
-                </friction>
-                <bounce>
-                    <restitution_coefficient>0.0</restitution_coefficient>
-                    <threshold>0.01</threshold>
-                </bounce>
-                <contact>
-                    <ode>
-                        <kp>1e5</kp>
-                        <max_vel>0.01</max_vel>
-                        <min_depth>0.001</min_depth>
+            <visual>
+            <material name="Black">
+                <color rgba="1.0 1.0 1.0 1.0"/>
+            </material>
+        </visual>
+        <collision>
+            <surface>
+                <friction>
+                    <ode>
+                        <mu>1.0</mu>
+                        <mu2>1.0</mu2>
+                    </ode>
+                </friction>
+                <bounce>
+                    <restitution_coefficient>0.0</restitution_coefficient>
+                    <threshold>0.01</threshold>
+                </bounce>
+                <contact>
+                    <ode>
+                        <kp>1e5</kp>
+                        <max_vel>0.1</max_vel>
+                        <min_depth>0.002</min_depth>
                     </ode>
                 </contact>
@@ -142,21 +152,26 @@
     </gazebo>
     <gazebo reference="FL_LOWER_LEG">
-        <collision>
-            <surface>
-                <friction>
-                    <ode>
-                        <mu>1.0</mu>
-                        <mu2>1.0</mu2>
-                    </ode>
-                </friction>
-                <bounce>
-                    <restitution_coefficient>0.0</restitution_coefficient>
-                    <threshold>0.01</threshold>
-                </bounce>
-                <contact>
-                    <ode>
-                        <kp>1e5</kp>
-                        <max_vel>0.01</max_vel>
-                        <min_depth>0.001</min_depth>
+            <visual>
+            <material name="Black">
+                <color rgba="1.0 1.0 1.0 1.0"/>
+            </material>
+        </visual>
+        <collision>
+            <surface>
+                <friction>
+                    <ode>
+                        <mu>1.0</mu>
+                        <mu2>1.0</mu2>
+                    </ode>
+                </friction>
+                <bounce>
+                    <restitution_coefficient>0.0</restitution_coefficient>
+                    <threshold>0.01</threshold>
+                </bounce>
+                <contact>
+                    <ode>
+                        <kp>1e5</kp>
+                        <max_vel>0.1</max_vel>
+                        <min_depth>0.002</min_depth>
                     </ode>
                 </contact>
@@ -165,21 +180,26 @@
     </gazebo>
     <gazebo reference="FR_UPPER_LEG">
-        <collision>
-            <surface>
-                <friction>
-                    <ode>
-                        <mu>1.0</mu>
-                        <mu2>1.0</mu2>
-                    </ode>
-                </friction>
-                <bounce>
-                    <restitution_coefficient>0.0</restitution_coefficient>
-                    <threshold>0.01</threshold>
-                </bounce>
-                <contact>
-                    <ode>
-                        <kp>1e5</kp>
-                        <max_vel>0.01</max_vel>
-                        <min_depth>0.001</min_depth>
+            <visual>
+            <material name="Black">
+                <color rgba="1.0 1.0 1.0 1.0"/>
+            </material>
+        </visual>
+        <collision>
+            <surface>
+                <friction>
+                    <ode>
+                        <mu>1.0</mu>
+                        <mu2>1.0</mu2>
+                    </ode>
+                </friction>
+                <bounce>
+                    <restitution_coefficient>0.0</restitution_coefficient>
+                    <threshold>0.01</threshold>
+                </bounce>
+                <contact>
+                    <ode>
+                        <kp>1e5</kp>
+                        <max_vel>0.1</max_vel>
+                        <min_depth>0.002</min_depth>
                     </ode>
                 </contact>
@@ -188,21 +208,26 @@
     </gazebo>
     <gazebo reference="FR_LOWER_LEG">
-        <collision>
-            <surface>
-                <friction>
-                    <ode>
-                        <mu>1.0</mu>
-                        <mu2>1.0</mu2>
-                    </ode>
-                </friction>
-                <bounce>
-                    <restitution_coefficient>0.0</restitution_coefficient>
-                    <threshold>0.01</threshold>
-                </bounce>
-                <contact>
-                    <ode>
-                        <kp>1e5</kp>
-                        <max_vel>0.01</max_vel>
-                        <min_depth>0.001</min_depth>
+            <visual>
+            <material name="Black">
+                <color rgba="1.0 1.0 1.0 1.0"/>
+            </material>
+        </visual>
+        <collision>
+            <surface>
+                <friction>
+                    <ode>
+                        <mu>1.0</mu>
+                        <mu2>1.0</mu2>
+                    </ode>
+                </friction>
+                <bounce>
+                    <restitution_coefficient>0.0</restitution_coefficient>
+                    <threshold>0.01</threshold>
+                </bounce>
+                <contact>
+                    <ode>
+                        <kp>1e5</kp>
+                        <max_vel>0.1</max_vel>
+                        <min_depth>0.002</min_depth>
                     </ode>
                 </contact>
@@ -211,21 +236,26 @@
     </gazebo>
     <gazebo reference="HL_UPPER_LEG">
-        <collision>
-            <surface>
-                <friction>
-                    <ode>
-                        <mu>1.0</mu>
-                        <mu2>1.0</mu2>
-                    </ode>
-                </friction>
-                <bounce>
-                    <restitution_coefficient>0.0</restitution_coefficient>
-                    <threshold>0.01</threshold>
-                </bounce>
-                <contact>
-                    <ode>
-                        <kp>1e5</kp>
-                        <max_vel>0.01</max_vel>
-                        <min_depth>0.001</min_depth>
+            <visual>
+            <material name="Black">
+                <color rgba="1.0 1.0 1.0 1.0"/>
+            </material>
+        </visual>
+        <collision>
+            <surface>
+                <friction>
+                    <ode>
+                        <mu>1.0</mu>
+                        <mu2>1.0</mu2>
+                    </ode>
+                </friction>
+                <bounce>
+                    <restitution_coefficient>0.0</restitution_coefficient>
+                    <threshold>0.01</threshold>
+                </bounce>
+                <contact>
+                    <ode>
+                        <kp>1e5</kp>
+                        <max_vel>0.1</max_vel>
+                        <min_depth>0.002</min_depth>
                     </ode>
                 </contact>
@@ -234,21 +264,26 @@
     </gazebo>
     <gazebo reference="HL_LOWER_LEG">
-        <collision>
-            <surface>
-                <friction>
-                    <ode>
-                        <mu>1.0</mu>
-                        <mu2>1.0</mu2>
-                    </ode>
-                </friction>
-                <bounce>
-                    <restitution_coefficient>0.0</restitution_coefficient>
-                    <threshold>0.01</threshold>
-                </bounce>
-                <contact>
-                    <ode>
-                        <kp>1e5</kp>
-                        <max_vel>0.01</max_vel>
-                        <min_depth>0.001</min_depth>
+            <visual>
+            <material name="Black">
+                <color rgba="1.0 1.0 1.0 1.0"/>
+            </material>
+        </visual>
+        <collision>
+            <surface>
+                <friction>
+                    <ode>
+                        <mu>1.0</mu>
+                        <mu2>1.0</mu2>
+                    </ode>
+                </friction>
+                <bounce>
+                    <restitution_coefficient>0.0</restitution_coefficient>
+                    <threshold>0.01</threshold>
+                </bounce>
+                <contact>
+                    <ode>
+                        <kp>1e5</kp>
+                        <max_vel>0.1</max_vel>
+                        <min_depth>0.002</min_depth>
                     </ode>
                 </contact>
@@ -257,21 +292,26 @@
     </gazebo>
 <gazebo reference="HR_UPPER_LEG">
-        <collision>
-            <surface>
-                <friction>
-                    <ode>
-                        <mu>1.0</mu>
-                        <mu2>1.0</mu2>
-                    </ode>
-                </friction>
-                <bounce>
-                    <restitution_coefficient>0.0</restitution_coefficient>
-                    <threshold>0.01</threshold>
-                </bounce>
-                <contact>
-                    <ode>
-                        <kp>1e5</kp>
-                        <max_vel>0.01</max_vel>
-                        <min_depth>0.001</min_depth>
+        <visual>
+            <material name="Black">
+                <color rgba="1.0 1.0 1.0 1.0"/>
+            </material>
+        </visual>
+        <collision>
+            <surface>
+                <friction>
+                    <ode>
+                        <mu>1.0</mu>
+                        <mu2>1.0</mu2>
+                    </ode>
+                </friction>
+                <bounce>
+                    <restitution_coefficient>0.0</restitution_coefficient>
+                    <threshold>0.01</threshold>
+                </bounce>
+                <contact>
+                    <ode>
+                        <kp>1e5</kp>
+                        <max_vel>0.1</max_vel>
+                        <min_depth>0.002</min_depth>
                     </ode>
                 </contact>
@@ -280,25 +320,51 @@
     </gazebo>
     <gazebo reference="HR_LOWER_LEG">
-        <collision>
-            <surface>
-                <friction>
-                    <ode>
-                        <mu>1.0</mu>
-                        <mu2>1.0</mu2>
-                    </ode>
-                </friction>
-                <bounce>
-                    <restitution_coefficient>0.0</restitution_coefficient>
-                    <threshold>0.01</threshold>
-                </bounce>
-                <contact>
-                    <ode>
-                        <kp>1e5</kp>
-                        <max_vel>0.01</max_vel>
-                        <min_depth>0.001</min_depth>
-                    </ode>
-                </contact>
-            </surface>
-        </collision>
-    </gazebo>
+            <visual>
+            <material name="Black">
+                <color rgba="1.0 1.0 1.0 1.0"/>
+            </material>
+        </visual>
+        <collision>
+            <surface>
+                <friction>
+                    <ode>
+                        <mu>1.0</mu>
+                        <mu2>1.0</mu2>
+                    </ode>
+                </friction>
+                <bounce>
+                    <restitution_coefficient>0.0</restitution_coefficient>
+                    <threshold>0.01</threshold>
+                </bounce>
+                <contact>
+                    <ode>
+                        <kp>1e5</kp>
+                        <max_vel>0.1</max_vel>
+                        <min_depth>0.002</min_depth>
+                    </ode>
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
Commit message: fall recovery

File: src/perrobot_description/urdf/gazebo.xacro (robot description, xacro)
@@ -96,9 +96,4 @@
     </transmission>
    <gazebo reference="base_link">
-        <visual>
-            <material name="Black">
-                <color rgba="1.0 1.0 1.0 1.0"/>
-            </material>
-        </visual>
         <collision>
             <surface>
@@ -124,9 +119,4 @@
     </gazebo>
     <gazebo reference="FL_UPPER_LEG">
-            <visual>
-            <material name="Black">
-                <color rgba="1.0 1.0 1.0 1.0"/>
-            </material>
-        </visual>
         <collision>
             <surface>
@@ -152,9 +142,4 @@
     </gazebo>
     <gazebo reference="FL_LOWER_LEG">
-            <visual>
-            <material name="Black">
-                <color rgba="1.0 1.0 1.0 1.0"/>
-            </material>
-        </visual>
         <collision>
             <surface>
@@ -180,9 +165,4 @@
     </gazebo>
     <gazebo reference="FR_UPPER_LEG">
-            <visual>
-            <material name="Black">
-                <color rgba="1.0 1.0 1.0 1.0"/>
-            </material>
-        </visual>
         <collision>
             <surface>
@@ -208,9 +188,4 @@
     </gazebo>
     <gazebo reference="FR_LOWER_LEG">
-            <visual>
-            <material name="Black">
-                <color rgba="1.0 1.0 1.0 1.0"/>
-            </material>
-        </visual>
         <collision>
             <surface>
@@ -236,9 +211,4 @@
     </gazebo>
     <gazebo reference="HL_UPPER_LEG">
-            <visual>
-            <material name="Black">
-                <color rgba="1.0 1.0 1.0 1.0"/>
-            </material>
-        </visual>
         <collision>
             <surface>
@@ -264,9 +234,4 @@
     </gazebo>
     <gazebo reference="HL_LOWER_LEG">
-            <visual>
-            <material name="Black">
-                <color rgba="1.0 1.0 1.0 1.0"/>
-            </material>
-        </visual>
         <collision>
             <surface>
@@ -292,9 +257,4 @@
     </gazebo>
 <gazebo reference="HR_UPPER_LEG">
-        <visual>
-            <material name="Black">
-                <color rgba="1.0 1.0 1.0 1.0"/>
-            </material>
-        </visual>
         <collision>
             <surface>
@@ -320,9 +280,4 @@
     </gazebo>
     <gazebo reference="HR_LOWER_LEG">
-            <visual>
-            <material name="Black">
-                <color rgba="1.0 1.0 1.0 1.0"/>
-            </material>
-        </visual>
         <collision>
             <surface>
@@ -356,5 +311,5 @@
       <topic>__default_topic__</topic>
       <plugin filename="libgazebo_ros_imu_sensor.so" name="imu_plugin">
-        <topicName>notspot_imu/base_link_orientation</topicName>
+        <topicName>perrobot/base_link_orientation</topicName>
         <bodyName>imu_link</bodyName>
         <updateRateHZ>15.0</updateRateHZ>

File: src/perrobot_description/urdf/leg.xacro (robot description, xacro)
@@ -13,5 +13,5 @@
   <xacro:property name="KFE_2_FOOT_y" value="${9.0 * 0.001}" />
   <xacro:property name="KFE_2_FOOT_z" value="${160.00 * 0.001}" />
-  <xacro:property name="effort_limit" value="1.7" />
+  <xacro:property name="effort_limit" value="2.7" />
   <!-- Macro defining solo leg. -->
   <xacro:macro name="leg" params="prefix is_front is_right has_side_motion
