Commit message: lets ggooo

File: src/perrobot_description/urdf/gazebo_12dof.xacro (robot description, xacro)
@@ -141,6 +141,6 @@
                 <friction>
                     <ode>
-                        <mu>3.0</mu>
-                        <mu2>3.0</mu2>
+                        <mu>1.0</mu>
+                        <mu2>1.0</mu2>
                     </ode>
                 </friction>
@@ -164,6 +164,6 @@
                 <friction>
                     <ode>
-                        <mu>3.0</mu>
-                        <mu2>3.0</mu2>
+                        <mu>1.0</mu>
+                        <mu2>1.0</mu2>
                     </ode>
                 </friction>
@@ -187,6 +187,6 @@
                 <friction>
                     <ode>
-                        <mu>3.0</mu>
-                        <mu2>3.0</mu2>
+                        <mu>1.0</mu>
+                        <mu2>1.0</mu2>
                     </ode>
                 </friction>
@@ -210,6 +210,6 @@
                 <friction>
                     <ode>
-                        <mu>3.0</mu>
-                        <mu2>3.0</mu2>
+                        <mu>1.0</mu>
+                        <mu2>1.0</mu2>
                     </ode>
                 </friction>
@@ -233,6 +233,6 @@
                 <friction>
                     <ode>
-                        <mu>3.0</mu>
-                        <mu2>3.0</mu2>
+                        <mu>1.0</mu>
+                        <mu2>1.0</mu2>
                     </ode>
                 </friction>
@@ -256,6 +256,6 @@
                 <friction>
                     <ode>
-                        <mu>3.0</mu>
-                        <mu2>3.0</mu2>
+                        <mu>1.0</mu>
+                        <mu2>1.0</mu2>
                     </ode>
                 </friction>
@@ -279,6 +279,6 @@
                 <friction>
                     <ode>
-                        <mu>3.0</mu>
-                        <mu2>3.0</mu2>
+                        <mu>1.0</mu>
+                        <mu2>1.0</mu2>
                     </ode>
                 </friction>
@@ -302,6 +302,6 @@
                 <friction>
                     <ode>
-                        <mu>3.0</mu>
-                        <mu2>3.0</mu2>
+                        <mu>1.0</mu>
+                        <mu2>1.0</mu2>
                     </ode>
                 </friction>
@@ -325,6 +325,6 @@
                 <friction>
                     <ode>
-                        <mu>3.0</mu>
-                        <mu2>3.0</mu2>
+                        <mu>1.0</mu>
+                        <mu2>1.0</mu2>
                     </ode>
                 </friction>
@@ -348,6 +348,6 @@
                 <friction>
                     <ode>
-                        <mu>3.0</mu>
-                        <mu2>3.0</mu2>
+                        <mu>1.0</mu>
+                        <mu2>1.0</mu2>
                     </ode>
                 </friction>
@@ -371,6 +371,6 @@
                 <friction>
                     <ode>
-                        <mu>3.0</mu>
-                        <mu2>3.0</mu2>
+                        <mu>1.0</mu>
+                        <mu2>1.0</mu2>
                     </ode>
                 </friction>
@@ -394,6 +394,6 @@
                 <friction>
                     <ode>
-                        <mu>3.0</mu>
-                        <mu2>3.0</mu2>
+                        <mu>1.0</mu>
+                        <mu2>1.0</mu2>
                     </ode>
                 </friction>
@@ -417,6 +417,6 @@
                 <friction>
                     <ode>
-                        <mu>3.0</mu>
-                        <mu2>3.0</mu2>
+                        <mu>1.0</mu>
+                        <mu2>1.0</mu2>
                     </ode>
                 </friction>

File: src/perrobot_description/urdf/leg.xacro (robot description, xacro)
@@ -13,5 +13,5 @@
   <xacro:property name="KFE_2_FOOT_y" value="${9.0 * 0.001}" />
   <xacro:property name="KFE_2_FOOT_z" value="${160.00 * 0.001}" />
-  <xacro:property name="effort_limit" value="2.4" />
+  <xacro:property name="effort_limit" value="1.8" />
   <xacro:property name="quater_pi" value="0.78539816339" />
   <!-- Macro defining solo leg. -->

Commit message: news

File: src/perrobot_description/urdf/gazebo_12dof.xacro (robot description, xacro)
@@ -1,4 +1,5 @@
 <?xml version="10.0"?>
 <robot xmlns:xacro="http://playerstage.sourceforge.net/gazebo/xmlschema/#interface" name="perrobot_12dof">
+    <xacro:property name="mechanicalReduction" value="5" />
   <gazebo>
     <plugin name="gazebo_ros_control" filename="libgazebo_ros_control.so">
@@ -23,5 +24,5 @@
         <actuator name="FL_HFE_actuator">
             <hardwareInterface>hardware_interface/EffortJointInterface</hardwareInterface>
-            <mechanicalReduction>5</mechanicalReduction>
+            <mechanicalReduction>"${mechanicalReduction}"</mechanicalReduction>
         </actuator>
     </transmission>
@@ -33,5 +34,5 @@
         <actuator name="FR_HFE_actuator">
             <hardwareInterface>hardware_interface/EffortJointInterface</hardwareInterface>
-            <mechanicalReduction>5</mechanicalReduction>
+            <mechanicalReduction>"${mechanicalReduction}"</mechanicalReduction>
         </actuator>
     </transmission>
@@ -43,5 +44,5 @@
         <actuator name="HL_HFE_actuator">
             <hardwareInterface>hardware_interface/EffortJointInterface</hardwareInterface>
-            <mechanicalReduction>5</mechanicalReduction>
+            <mechanicalReduction>"${mechanicalReduction}"</mechanicalReduction>
         </actuator>
     </transmission>
@@ -53,5 +54,5 @@
         <actuator name="HR_HFE_actuator">
             <hardwareInterface>hardware_interface/EffortJointInterface</hardwareInterface>
-            <mechanicalReduction>5</mechanicalReduction>
+            <mechanicalReduction>"${mechanicalReduction}"</mechanicalReduction>
         </actuator>
     </transmission>
@@ -63,5 +64,5 @@
         <actuator name="FL_KFE_actuator">
             <hardwareInterface>hardware_interface/EffortJointInterface</hardwareInterface>
-            <mechanicalReduction>5</mechanicalReduction>
+            <mechanicalReduction>"${mechanicalReduction}"</mechanicalReduction>
         </actuator>
     </transmission>
@@ -73,5 +74,5 @@
         <actuator name="FR_KFE_actuator">
             <hardwareInterface>hardware_interface/EffortJointInterface</hardwareInterface>
-            <mechanicalReduction>5</mechanicalReduction>
+            <mechanicalReduction>"${mechanicalReduction}"</mechanicalReduction>
         </actuator>
     </transmission>
@@ -83,5 +84,5 @@
         <actuator name="HL_KFE_actuator">
             <hardwareInterface>hardware_interface/EffortJointInterface</hardwareInterface>
-            <mechanicalReduction>5</mechanicalReduction>
+            <mechanicalReduction>"${mechanicalReduction}"</mechanicalReduction>
         </actuator>
     </transmission>
@@ -93,5 +94,5 @@
         <actuator name="HR_KFE_actuator">
             <hardwareInterface>hardware_interface/EffortJointInterface</hardwareInterface>
-            <mechanicalReduction>5</mechanicalReduction>
+            <mechanicalReduction>"${mechanicalReduction}"</mechanicalReduction>
         </actuator>
     </transmission>
@@ -103,5 +104,5 @@
         <actuator name="HR_HAA_actuator">
             <hardwareInterface>hardware_interface/EffortJointInterface</hardwareInterface>
-            <mechanicalReduction>5</mechanicalReduction>
+            <mechanicalReduction>"${mechanicalReduction}"</mechanicalReduction>
         </actuator>
     </transmission>
@@ -113,5 +114,5 @@
         <actuator name="HL_HAA_actuator">
             <hardwareInterface>hardware_interface/EffortJointInterface</hardwareInterface>
-            <mechanicalReduction>5</mechanicalReduction>
+            <mechanicalReduction>"${mechanicalReduction}"</mechanicalReduction>
         </actuator>
     </transmission>
@@ -123,5 +124,5 @@
         <actuator name="FR_HAA_actuator">
             <hardwareInterface>hardware_interface/EffortJointInterface</hardwareInterface>
-            <mechanicalReduction>5</mechanicalReduction>
+            <mechanicalReduction>"${mechanicalReduction}"</mechanicalReduction>
         </actuator>
     </transmission>
@@ -133,5 +134,5 @@
         <actuator name="FL_HAA_actuator">
             <hardwareInterface>hardware_interface/EffortJointInterface</hardwareInterface>
-            <mechanicalReduction>5</mechanicalReduction>
+            <mechanicalReduction>"${mechanicalReduction}"</mechanicalReduction>
         </actuator>
     </transmission>

File: src/perrobot_description/urdf/leg.xacro (robot description, xacro)
@@ -13,5 +13,5 @@
   <xacro:property name="KFE_2_FOOT_y" value="${9.0 * 0.001}" />
   <xacro:property name="KFE_2_FOOT_z" value="${160.00 * 0.001}" />
-  <xacro:property name="effort_limit" value="1.8" />
+  <xacro:property name="effort_limit" value="1.4" />
   <xacro:property name="quater_pi" value="0.78539816339" />
   <!-- Macro defining solo leg. -->
