Commit message: something new

File: src/perrobot_description/urdf/leg.xacro (robot description, xacro)
@@ -13,5 +13,5 @@
   <xacro:property name="KFE_2_FOOT_y" value="${9.0 * 0.001}" />
   <xacro:property name="KFE_2_FOOT_z" value="${160.00 * 0.001}" />
-  <xacro:property name="effort_limit" value="1.4" />
+  <xacro:property name="effort_limit" value="1.7" />
   <!-- Macro defining solo leg. -->
   <xacro:macro name="leg" params="prefix is_front is_right has_side_motion

Commit message: addind 12dof - work in progress

File: src/perrobot_description/urdf/leg.xacro (robot description, xacro)
@@ -1,5 +1,5 @@
 <?xml version="1.0"?>
-<robot xmlns:xacro="http://playerstage.sourceforge.net/gazebo/xmlschema/#interface" name="solo">
-  <!-- See https://github.com/open-dynamic-robot-initiative/open_robot_actuator_hardware/blob/master/mechanics/perrobot_description_12dof_v1/README.md#quadruped-robot-12dof-v1 -->
+<robot xmlns:xacro="http://playerstage.sourceforge.net/gazebo/xmlschema/#interface" name="perrobot_12dof">
+  <!-- See https://github.com/open-dynamic-robot-initiative/open_robot_actuator_hardware/blob/master/mechanics/perrobot_12dof_description_12dof_v1/README.md#quadruped-robot-12dof-v1 -->
   <!-- These are absoulte distance value, the sign are decided below -->
   <xacro:property name="base_2_HAA_x" value="${214.10 * 0.001}" />
@@ -14,4 +14,5 @@
   <xacro:property name="KFE_2_FOOT_z" value="${160.00 * 0.001}" />
   <xacro:property name="effort_limit" value="2.7" />
+  <xacro:property name="quater_pi" value="0.78539816339" />
   <!-- Macro defining solo leg. -->
   <xacro:macro name="leg" params="prefix is_front is_right has_side_motion
@@ -21,5 +22,5 @@
         <parent link="base_link"/>
         <child link="${prefix}_SHOULDER"/>
-        <limit effort="${effort_limit}" lower="-10" upper="10" velocity="1000"/>
+        <limit effort="${effort_limit}" lower="-${quater_pi}" upper="${quater_pi}" velocity="1000"/>
         <!-- joints rotates around the x-axis -->
         <axis xyz="1 0 0"/>
@@ -51,5 +52,5 @@
                     <origin xyz="0.01950 0 0" rpy="0 0 0" />
                     <geometry>
-                        <mesh filename="package://perrobot_description/meshes/solo12/solo12_hip_fe_fl.${mesh_ext}"/>
+                        <mesh filename="package://perrobot_12dof_description/meshes/solo12/solo12_hip_fe_fl.${mesh_ext}"/>
                     </geometry>
                 </xacro:if>
@@ -57,5 +58,5 @@
                     <origin xyz="-0.01950 0 0" rpy="0 0 0" />
                     <geometry>
-                        <mesh filename="package://perrobot_description/meshes/solo12/solo12_hip_fe_hl.${mesh_ext}"/>
+                        <mesh filename="package://perrobot_12dof_description/meshes/solo12/solo12_hip_fe_hl.${mesh_ext}"/>
                     </geometry>
                 </xacro:unless>
@@ -65,5 +66,5 @@
                     <origin xyz="0.01950 0 0" rpy="0 0 0" />
                     <geometry>
-                        <mesh filename="package://perrobot_description/meshes/solo12/solo12_hip_fe_fr.${mesh_ext}"/>
+                        <mesh filename="package://perrobot_12dof_description/meshes/solo12/solo12_hip_fe_fr.${mesh_ext}"/>
                     </geometry>
                 </xacro:if>
@@ -71,5 +72,5 @@
                     <origin xyz="-0.01950 0 0" rpy="0 0 0" />
                     <geometry>
-                        <mesh filename="package://perrobot_description/meshes/solo12/solo12_hip_fe_hr.${mesh_ext}"/>
+                        <mesh filename="package://perrobot_12dof_description/meshes/solo12/solo12_hip_fe_hr.${mesh_ext}"/>
                     </geometry>
                 </xacro:unless>
@@ -85,5 +86,5 @@
                     <origin xyz="0.01950 0 0" rpy="0 0 0" />
                     <geometry>
-                        <mesh filename="package://perrobot_description/meshes/solo12/solo12_hip_fe_fl.${mesh_ext}"/>
+                        <mesh filename="package://perrobot_12dof_description/meshes/solo12/solo12_hip_fe_fl.${mesh_ext}"/>
                     </geometry>
                 </xacro:if>
@@ -91,5 +92,5 @@
                     <origin xyz="-0.01950 0 0" rpy="0 0 0" />
                     <geometry>
-                        <mesh filename="package://perrobot_description/meshes/solo12/solo12_hip_fe_hl.${mesh_ext}"/>
+                        <mesh filename="package://perrobot_12dof_description/meshes/solo12/solo12_hip_fe_hl.${mesh_ext}"/>
                     </geometry>
                 </xacro:unless>
@@ -99,5 +100,5 @@
                     <origin xyz="0.01950 0 0" rpy="0 0 0" />
                     <geometry>
-                        <mesh filename="package://perrobot_description/meshes/solo12/solo12_hip_fe_fr.${mesh_ext}"/>
+                        <mesh filename="package://perrobot_12dof_description/meshes/solo12/solo12_hip_fe_fr.${mesh_ext}"/>
                     </geometry>
                 </xacro:if>
@@ -105,5 +106,5 @@
                     <origin xyz="-0.01950 0 0" rpy="0 0 0" />
                     <geometry>
-                        <mesh filename="package://perrobot_description/meshes/solo12/solo12_hip_fe_hr.${mesh_ext}"/>
+                        <mesh filename="package://perrobot_12dof_description/meshes/solo12/solo12_hip_fe_hr.${mesh_ext}"/>
                     </geometry>
                 </xacro:unless>
@@ -232,8 +233,8 @@
         <geometry>
           <xacro:unless value="${is_right}">
-            <mesh filename="package://perrobot_description/meshes/without_foot/solo_upper_leg_left_side.${mesh_ext}"/>
-          </xacro:unless>
-          <xacro:if value="${is_right}">
-            <mesh filename="package://perrobot_description/meshes/without_foot/solo_upper_leg_right_side.${mesh_ext}"/>
+            <mesh filename="package://perrobot_12dof_description/meshes/without_foot/solo_upper_leg_left_side.${mesh_ext}"/>
+          </xacro:unless>
+          <xacro:if value="${is_right}">
+            <mesh filename="package://perrobot_12dof_description/meshes/without_foot/solo_upper_leg_right_side.${mesh_ext}"/>
           </xacro:if>
         </geometry>
@@ -247,8 +248,8 @@
         <geometry>
           <xacro:unless value="${is_right}">
-            <mesh filename="package://perrobot_description/meshes/without_foot/solo_upper_leg_left_side.${mesh_ext}"/>
-          </xacro:unless>
-          <xacro:if value="${is_right}">
-            <mesh filename="package://perrobot_description/meshes/without_foot/solo_upper_leg_right_side.${mesh_ext}"/>
+            <mesh filename="package://perrobot_12dof_description/meshes/without_foot/solo_upper_leg_left_side.${mesh_ext}"/>
+          </xacro:unless>
+          <xacro:if value="${is_right}">
+            <mesh filename="package://perrobot_12dof_description/meshes/without_foot/solo_upper_leg_right_side.${mesh_ext}"/>
           </xacro:if>
         </geometry>
@@ -317,8 +318,8 @@
         <geometry>
           <xacro:unless value="${is_right}">
-            <mesh filename="package://perrobot_description/meshes/without_foot/solo_lower_leg_v2_left_side.${mesh_ext}"/>
-          </xacro:unless>
-          <xacro:if value="${is_right}">
-            <mesh filename="package://perrobot_description/meshes/without_foot/solo_lower_leg_v2_right_side.${mesh_ext}"/>
+            <mesh filename="package://perrobot_12dof_description/meshes/without_foot/solo_lower_leg_v2_left_side.${mesh_ext}"/>
+          </xacro:unless>
+          <xacro:if value="${is_right}">
+            <mesh filename="package://perrobot_12dof_description/meshes/without_foot/solo_lower_leg_v2_right_side.${mesh_ext}"/>
           </xacro:if>
         </geometry>
@@ -332,8 +333,8 @@
         <geometry>
           <xacro:unless value="${is_right}">
-            <mesh filename="package://perrobot_description/meshes/without_foot/solo_lower_leg_v2_left_side.${mesh_ext}"/>
-          </xacro:unless>
-          <xacro:if value="${is_right}">
-            <mesh filename="package://perrobot_description/meshes/without_foot/solo_lower_leg_v2_right_side.${mesh_ext}"/>
+            <mesh filename="package://perrobot_12dof_description/meshes/without_foot/solo_lower_leg_v2_left_side.${mesh_ext}"/>
+          </xacro:unless>
+          <xacro:if value="${is_right}">
+            <mesh filename="package://perrobot_12dof_description/meshes/without_foot/solo_lower_leg_v2_right_side.${mesh_ext}"/>
           </xacro:if>
         </geometry>

File: src/perrobot_description/urdf/solo12.urdf.xacro (robot description, xacro)
@@ -1,4 +1,4 @@
 <?xml version="1.0" ?>
-<robot name="solo"
+<robot name="perrobot_12dof"
   xmlns:controller="http://playerstage.sourceforge.net/gazebo/xmlschema/#controller"
   xmlns:interface="http://playerstage.sourceforge.net/gazebo/xmlschema/#interface"
@@ -9,5 +9,5 @@
   <xacro:property name="opacity" value="1.0" />
   <xacro:property name="mesh_ext" value="stl" />
-  <!-- This file is based on: https://github.com/open-dynamic-robot-initiative/open_robot_actuator_hardware/blob/master/mechanics/perrobot_description_12dof_v1/README.md#quadruped-robot-12dof-v1 -->
+  <!-- This file is based on: https://github.com/open-dynamic-robot-initiative/open_robot_actuator_hardware/blob/master/mechanics/perrobot_12dofion_12dof_v1/README.md#quadruped-robot-12dof-v1 -->
   <link name="base_link">
     <!-- BASE LINK INERTIAL -->
@@ -25,5 +25,5 @@
         <origin xyz="0 0 0" rpy="0 0 0" />
         <geometry>
-          <mesh filename="package://perrobot_description/meshes/solo12/solo_12_base.${mesh_ext}"/>
+          <mesh filename="package://perrobot_12dof_description/meshes/solo12/solo_12_base.${mesh_ext}"/>
         </geometry>
         <material name="${color_name}">
@@ -35,5 +35,5 @@
         <origin xyz="0 0 0" rpy="0 0 0" />
         <geometry>
-          <mesh filename="package://perrobot_description/meshes/solo12/solo_12_base.${mesh_ext}"/>
+          <mesh filename="package://perrobot_12dof_description/meshes/solo12/solo_12_base.${mesh_ext}"/>
         </geometry>
         <material name="${color_name}">
@@ -49,4 +49,6 @@
   <!-- Include the legs -->
   <xacro:include filename="leg.xacro"/>
+  <!-- Include gazebo plugins and physics -->
+  <xacro:include filename="gazebo_12dof.xacro"/>
   <!-- Include the front left leg -->
   <xacro:leg

Commit message: description package corrected

File: src/perrobot_description/urdf/leg.xacro (robot description, xacro)
@@ -1,5 +1,5 @@
 <?xml version="1.0"?>
 <robot xmlns:xacro="http://playerstage.sourceforge.net/gazebo/xmlschema/#interface" name="perrobot_12dof">
-  <!-- See https://github.com/open-dynamic-robot-initiative/open_robot_actuator_hardware/blob/master/mechanics/perrobot_12dof_description_12dof_v1/README.md#quadruped-robot-12dof-v1 -->
+  <!-- See https://github.com/open-dynamic-robot-initiative/open_robot_actuator_hardware/blob/master/mechanics/perrobot_description_12dof_v1/README.md#quadruped-robot-12dof-v1 -->
   <!-- These are absoulte distance value, the sign are decided below -->
   <xacro:property name="base_2_HAA_x" value="${214.10 * 0.001}" />
@@ -13,5 +13,5 @@
   <xacro:property name="KFE_2_FOOT_y" value="${9.0 * 0.001}" />
   <xacro:property name="KFE_2_FOOT_z" value="${160.00 * 0.001}" />
-  <xacro:property name="effort_limit" value="2.7" />
+  <xacro:property name="effort_limit" value="2.4" />
   <xacro:property name="quater_pi" value="0.78539816339" />
   <!-- Macro defining solo leg. -->
@@ -52,5 +52,5 @@
                     <origin xyz="0.01950 0 0" rpy="0 0 0" />
                     <geometry>
-                        <mesh filename="package://perrobot_12dof_description/meshes/solo12/solo12_hip_fe_fl.${mesh_ext}"/>
+                        <mesh filename="package://perrobot_description/meshes/solo12/solo12_hip_fe_fl.${mesh_ext}"/>
                     </geometry>
                 </xacro:if>
@@ -58,5 +58,5 @@
                     <origin xyz="-0.01950 0 0" rpy="0 0 0" />
                     <geometry>
-                        <mesh filename="package://perrobot_12dof_description/meshes/solo12/solo12_hip_fe_hl.${mesh_ext}"/>
+                        <mesh filename="package://perrobot_description/meshes/solo12/solo12_hip_fe_hl.${mesh_ext}"/>
                     </geometry>
                 </xacro:unless>
@@ -66,5 +66,5 @@
                     <origin xyz="0.01950 0 0" rpy="0 0 0" />
                     <geometry>
-                        <mesh filename="package://perrobot_12dof_description/meshes/solo12/solo12_hip_fe_fr.${mesh_ext}"/>
+                        <mesh filename="package://perrobot_description/meshes/solo12/solo12_hip_fe_fr.${mesh_ext}"/>
                     </geometry>
                 </xacro:if>
@@ -72,5 +72,5 @@
                     <origin xyz="-0.01950 0 0" rpy="0 0 0" />
                     <geometry>
-                        <mesh filename="package://perrobot_12dof_description/meshes/solo12/solo12_hip_fe_hr.${mesh_ext}"/>
+                        <mesh filename="package://perrobot_description/meshes/solo12/solo12_hip_fe_hr.${mesh_ext}"/>
                     </geometry>
                 </xacro:unless>
@@ -86,5 +86,5 @@
                     <origin xyz="0.01950 0 0" rpy="0 0 0" />
                     <geometry>
-                        <mesh filename="package://perrobot_12dof_description/meshes/solo12/solo12_hip_fe_fl.${mesh_ext}"/>
+                        <mesh filename="package://perrobot_description/meshes/solo12/solo12_hip_fe_fl.${mesh_ext}"/>
                     </geometry>
                 </xacro:if>
@@ -92,5 +92,5 @@
                     <origin xyz="-0.01950 0 0" rpy="0 0 0" />
                     <geometry>
-                        <mesh filename="package://perrobot_12dof_description/meshes/solo12/solo12_hip_fe_hl.${mesh_ext}"/>
+                        <mesh filename="package://perrobot_description/meshes/solo12/solo12_hip_fe_hl.${mesh_ext}"/>
                     </geometry>
                 </xacro:unless>
@@ -100,5 +100,5 @@
                     <origin xyz="0.01950 0 0" rpy="0 0 0" />
                     <geometry>
-                        <mesh filename="package://perrobot_12dof_description/meshes/solo12/solo12_hip_fe_fr.${mesh_ext}"/>
+                        <mesh filename="package://perrobot_description/meshes/solo12/solo12_hip_fe_fr.${mesh_ext}"/>
                     </geometry>
                 </xacro:if>
@@ -106,5 +106,5 @@
                     <origin xyz="-0.01950 0 0" rpy="0 0 0" />
                     <geometry>
-                        <mesh filename="package://perrobot_12dof_description/meshes/solo12/solo12_hip_fe_hr.${mesh_ext}"/>
+                        <mesh filename="package://perrobot_description/meshes/solo12/solo12_hip_fe_hr.${mesh_ext}"/>
                     </geometry>
                 </xacro:unless>
@@ -233,8 +233,8 @@
         <geometry>
           <xacro:unless value="${is_right}">
-            <mesh filename="package://perrobot_12dof_description/meshes/without_foot/solo_upper_leg_left_side.${mesh_ext}"/>
-          </xacro:unless>
-          <xacro:if value="${is_right}">
-            <mesh filename="package://perrobot_12dof_description/meshes/without_foot/solo_upper_leg_right_side.${mesh_ext}"/>
+            <mesh filename="package://perrobot_description/meshes/without_foot/solo_upper_leg_left_side.${mesh_ext}"/>
+          </xacro:unless>
+          <xacro:if value="${is_right}">
+            <mesh filename="package://perrobot_description/meshes/without_foot/solo_upper_leg_right_side.${mesh_ext}"/>
           </xacro:if>
         </geometry>
@@ -248,8 +248,8 @@
         <geometry>
           <xacro:unless value="${is_right}">
-            <mesh filename="package://perrobot_12dof_description/meshes/without_foot/solo_upper_leg_left_side.${mesh_ext}"/>
-          </xacro:unless>
-          <xacro:if value="${is_right}">
-            <mesh filename="package://perrobot_12dof_description/meshes/without_foot/solo_upper_leg_right_side.${mesh_ext}"/>
+            <mesh filename="package://perrobot_description/meshes/without_foot/solo_upper_leg_left_side.${mesh_ext}"/>
+          </xacro:unless>
+          <xacro:if value="${is_right}">
+            <mesh filename="package://perrobot_description/meshes/without_foot/solo_upper_leg_right_side.${mesh_ext}"/>
           </xacro:if>
         </geometry>
@@ -318,8 +318,8 @@
         <geometry>
           <xacro:unless value="${is_right}">
-            <mesh filename="package://perrobot_12dof_description/meshes/without_foot/solo_lower_leg_v2_left_side.${mesh_ext}"/>
-          </xacro:unless>
-          <xacro:if value="${is_right}">
-            <mesh filename="package://perrobot_12dof_description/meshes/without_foot/solo_lower_leg_v2_right_side.${mesh_ext}"/>
+            <mesh filename="package://perrobot_description/meshes/without_foot/solo_lower_leg_v2_left_side.${mesh_ext}"/>
+          </xacro:unless>
+          <xacro:if value="${is_right}">
+            <mesh filename="package://perrobot_description/meshes/without_foot/solo_lower_leg_v2_right_side.${mesh_ext}"/>
           </xacro:if>
         </geometry>
@@ -333,8 +333,8 @@
         <geometry>
           <xacro:unless value="${is_right}">
-            <mesh filename="package://perrobot_12dof_description/meshes/without_foot/solo_lower_leg_v2_left_side.${mesh_ext}"/>
-          </xacro:unless>
-          <xacro:if value="${is_right}">
-            <mesh filename="package://perrobot_12dof_description/meshes/without_foot/solo_lower_leg_v2_right_side.${mesh_ext}"/>
+            <mesh filename="package://perrobot_description/meshes/without_foot/solo_lower_leg_v2_left_side.${mesh_ext}"/>
+          </xacro:unless>
+          <xacro:if value="${is_right}">
+            <mesh filename="package://perrobot_description/meshes/without_foot/solo_lower_leg_v2_right_side.${mesh_ext}"/>
           </xacro:if>
         </geometry>

File: src/perrobot_description/urdf/solo12.urdf.xacro (robot description, xacro)
@@ -25,5 +25,5 @@
         <origin xyz="0 0 0" rpy="0 0 0" />
         <geometry>
-          <mesh filename="package://perrobot_12dof_description/meshes/solo12/solo_12_base.${mesh_ext}"/>
+          <mesh filename="package://perrobot_description/meshes/solo12/solo_12_base.${mesh_ext}"/>
         </geometry>
         <material name="${color_name}">
@@ -35,5 +35,5 @@
         <origin xyz="0 0 0" rpy="0 0 0" />
         <geometry>
-          <mesh filename="package://perrobot_12dof_description/meshes/solo12/solo_12_base.${mesh_ext}"/>
+          <mesh filename="package://perrobot_description/meshes/solo12/solo_12_base.${mesh_ext}"/>
         </geometry>
         <material name="${color_name}">

Commit message: changes to leg.xacro legs limits back to -2pi 2pi

File: src/perrobot_description/urdf/leg.xacro (robot description, xacro)
@@ -14,4 +14,6 @@
   <xacro:property name="KFE_2_FOOT_z" value="${160.00 * 0.001}" />
   <xacro:property name="effort_limit" value="1.4" />
+  <xacro:property name="plus_2_pi" value="${2 * 22 / 7}" />
+  <xacro:property name="minus_2_pi" value="${-2 * 22 / 7}" />
   <xacro:property name="quater_pi" value="0.78539816339" />
   <!-- Macro defining solo leg. -->
@@ -153,5 +155,5 @@
         <parent link="${prefix}_SHOULDER"/>
         <child link="${prefix}_UPPER_LEG"/>
-        <limit effort="${effort_limit}" lower="-10" upper="10" velocity="1000"/>
+        <limit effort="${effort_limit}" lower="${minus_2_pi}" upper="${plus_2_pi}" velocity="1000"/>
         <!-- joints rotates around the y-axis -->
         <axis xyz="0 1 0"/>
@@ -182,5 +184,5 @@
         <parent link="base_link"/>
         <child link="${prefix}_UPPER_LEG"/>
-        <limit effort="${effort_limit}" lower="-10" upper="10" velocity="1000"/>
+        <limit effort="${effort_limit}" lower="${minus_2_pi}" upper="${plus_2_pi}" velocity="1000"/>
         <!-- joints rotates around the y-axis -->
         <axis xyz="0 1 0"/>
@@ -268,5 +270,5 @@
       <parent link="${prefix}_UPPER_LEG"/>
       <child link="${prefix}_LOWER_LEG"/>
-      <limit effort="${effort_limit}" lower="-10" upper="10" velocity="1000"/>
+      <limit effort="${effort_limit}" lower="${minus_2_pi}" upper="${plus_2_pi}" velocity="1000"/>
       <!-- joints rotates around the y-axis -->
       <axis xyz="0 1 0"/>
@@ -363,5 +365,5 @@
       </xacro:if>
       <!-- Limits -->
-      <limit effort="${effort_limit}" lower="-10" upper="10" velocity="1000"/>
+      <limit effort="${effort_limit}" lower="${minus_2_pi}" upper="${plus_2_pi}" velocity="1000"/>
       <!-- pybullet simulation parameters -->
       <dynamics damping="0.0" friction="0.0"/>
